File: pcb/ASBF.kicad_pcb (KiCad board)
At the start: 2 copper layers, 72 parts, among them J1 Conn_01x02, J10 Conn_01x01, J11 Conn_01x03, J12 Conn_01x03, J13 Conn_01x03, J14 Conn_01x02, J15 Conn_01x03, J16 Conn_01x02, J2 Screw_Terminal_01x02, J3 Screw_Terminal_01x03, J4 Conn_02x24_Counter_Clockwise, J5 Conn_01x03, J6 Conn_01x02, J7 Conn_01x13, J8 Conn_01x02, J9 Conn_01x02, U1 LMH6702MF, U2 ADC08060, U3 DAC5662A

Commit message: 1ra correcciones segun revision 1ra
Parts:
- C1, C11, C14, C15, C18, C19, C2, C20, C21, C22, C23, C24, C3, C5, C6, C7, C8: footprint Capacitor_THT:C_Disc_D3.0mm_W1.6mm_P2.50mm -> Resistor_SMD:R_0805_2012Metric
- C10, C12, C16, C17, C4, C9: footprint Capacitor_THT:CP_Radial_D4.0mm_P1.50mm -> Resistor_SMD:R_0805_2012Metric
- R1, R10, R11, R12, R13, R14, R15, R16, R17, R18, R19, R2, R20, R21, R22, R3, R4, R5, R6, R7, R8, R9: footprint Resistor_THT:R_Axial_DIN0207_L6.3mm_D2.5mm_P7.62mm_Horizontal -> Resistor_SMD:R_1206_3216Metric
- moved J1 196.3 mm to (24.1, 92.7)
- moved R17 190.0 mm to (259.4, 64.5)
- moved R14 187.8 mm to (246.8, 73.9)
- moved C18 185.3 mm to (253.8, 77.0)
- moved R16 182.3 mm to (244.4, 78.2)
- moved C15 182.3 mm to (264.4, 64.3)
- moved R18 174.1 mm to (239.8, 85.4)
- moved J3 173.6 mm to (24.1, 29.2), turned to 270 degrees
- moved J2 171.8 mm to (24.1, 52.1), turned to 270 degrees
- moved J10 171.4 mm to (258.9, 68.4)
- moved C23 170.4 mm to (249.4, 79.9)
- moved C24 169.3 mm to (244.8, 84.6)
- moved R15 168.0 mm to (230.9, 91.2)
- moved C17 166.6 mm to (263.4, 67.6)
- moved R20 166.2 mm to (252.4, 73.9)
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
Commit message: Realizado de PCB
Parts:
- added H1: MountingHole, MountingHole:MountingHole_2.5mm, B.Cu at (102.7, 120.6)
- added H2: MountingHole, MountingHole:MountingHole_2.5mm, B.Cu at (207.4, 44.0)
- added J17: Screw_Terminal_01x03, TerminalBlock:TerminalBlock_bornier-3_P5.08mm, F.Cu at (142.6, 118.5)
- C1, C11, C14, C15, C18, C19, C2, C20, C22, C24, C3, C5, C6, C7, C8, R1, R10, R11, R12, R13, R14, R15, R16, R17, R18, R19, R2, R20, R21, R22, R3, R4, R5, R6, R7, R8, R9, TR1, TR2, U1, U3: moved to B.Cu
- C10, C12, C16, C17, C4, C9: footprint Resistor_SMD:R_0805_2012Metric -> Capacitor_THT:CP_Radial_D4.0mm_P1.50mm
- C21, C23: value 100NF -> 100nf; moved to B.Cu
- U2: value ADC08060 -> ADC080200; moved to B.Cu
- moved J3 107.6 mm to (130.0, 48.5), turned to 180 degrees
- moved J10 95.6 mm to (167.9, 97.8)
- moved C17 95.5 mm to (168.4, 57.6), turned to 90 degrees
- moved C15 90.6 mm to (174.1, 56.5), turned to 90 degrees
- moved L2 89.3 mm to (163.7, 114.5), turned to 90 degrees
- moved J2 87.9 mm to (112.0, 48.5), turned to 180 degrees
- moved R20 87.7 mm to (175.0, 115.2), turned to 90 degrees
- moved R17 86.2 mm to (186.8, 111.1), turned to 270 degrees
- moved J1 85.7 mm to (109.5, 84.9)
- moved J12 83.6 mm to (171.4, 120.7), turned to 270 degrees
- moved J11 82.5 mm to (167.8, 105.8), turned to 90 degrees
- moved L1 81.2 mm to (118.6, 117.5)
- moved C12 78.6 mm to (181.5, 116.6), turned to 90 degrees
- moved C18 77.3 mm to (187.0, 115.7), turned to 90 degrees
- moved C22 74.7 mm to (167.9, 101.7), turned to 270 degrees
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Connections:
- J1 pad 1: GND -> Net-(J1-Pad1)
- J1 pad 2: Net-(J1-Pad2) -> GND
- J3 pad 1: GND -> +5V
- J3 pad 3: +5V -> GND
- J4 pad 10: /ADC/PWR_DWN -> /FPGA_Conector/W3
- J4 pad 11: /ADC/CLK -> /FPGA_Conector/V3
- J4 pad 15: /FPGA_Conector/V5 -> /ADC/D8
- J4 pad 16: /FPGA_Conector/W4 -> /ADC/D7
- J4 pad 17: /FPGA_Conector/U5 -> /ADC/D5
- J4 pad 18: /FPGA_Conector/U2 -> /ADC/D4
- J4 pad 19: /FPGA_Conector/W6 -> /ADC/D3
- J4 pad 2: /ADC/D0 -> /FPGA_Conector/R3
- J4 pad 20: /FPGA_Conector/U3 -> /ADC/D2
- J4 pad 21: /FPGA_Conector/U7 -> /ADC/D1
- J4 pad 22: /FPGA_Conector/W7 -> /ADC/D0
- J4 pad 23: /FPGA_Conector/U8 -> /ADC/CLK
- J4 pad 24: /FPGA_Conector/V8 -> /ADC/PWR_DWN
- J4 pad 3: /ADC/D1 -> /FPGA_Conector/T3
- J4 pad 34: /FPGA_Conector/J3 -> /DAC/DA9
- J4 pad 35: /DAC/ClkA -> /DAC/DA8
- J4 pad 36: /DAC/DA0 -> /DAC/DA7
- J4 pad 37: /DAC/DA1 -> /DAC/DA6
- J4 pad 38: /DAC/DA2 -> /DAC/DA5
- J4 pad 39: /DAC/DA3 -> /DAC/DA4
- J4 pad 4: /ADC/D2 -> /FPGA_Conector/R2
- J4 pad 40: /DAC/DA4 -> /DAC/DA3
- J4 pad 41: /DAC/DA5 -> /DAC/DA2
- J4 pad 42: /DAC/DA6 -> /DAC/DA1
- J4 pad 43: /DAC/DA7 -> /DAC/DA0
- J4 pad 44: /DAC/DA8 -> /DAC/ClkA
- J4 pad 45: /DAC/DA9 -> /FPGA_Conector/N1
- J4 pad 46: /DAC/DA10 -> Net-(J17-Pad2)
- J4 pad 47: /DAC/DA11 -> Net-(J17-Pad1)
- J4 pad 5: /ADC/D3 -> /FPGA_Conector/T1
- J4 pad 6: /ADC/D4 -> /FPGA_Conector/T2
- J4 pad 7: /ADC/D5 -> /FPGA_Conector/U1
- J4 pad 8: /ADC/D7 -> /FPGA_Conector/W2
- J4 pad 9: /ADC/D8 -> /FPGA_Conector/V2
- R1 pad 2: Net-(J1-Pad2) -> Net-(J1-Pad1)
- R3 pad 1: Net-(J1-Pad2) -> Net-(J1-Pad1)
- RV2 pad 1: Net-(R6-Pad2) -> Net-(R2-Pad1)
- RV2 pad 3: Net-(R2-Pad1) -> Net-(R6-Pad2)
- U2 pad 13: /ADC/D0 -> /ADC/D8
- U2 pad 14: /ADC/D1 -> /ADC/D7
- U2 pad 15: /ADC/D2 -> /ADC/D5
- U2 pad 16: /ADC/D3 -> /ADC/D4
- U2 pad 19: /ADC/D4 -> /ADC/D3
- U2 pad 20: /ADC/D5 -> /ADC/D2
- U2 pad 21: /ADC/D7 -> /ADC/D1
- U2 pad 22: /ADC/D8 -> /ADC/D0
- U3 pad 1: /DAC/DA11 -> /FPGA_Conector/B15
- U3 pad 2: /DAC/DA10 -> /FPGA_Conector/A14
Routing:
- net GND: track 0.00 -> 652.3 mm, vias 0 -> 12
- net +3V3: track 0.00 -> 277.1 mm
- net Net-(J17-Pad1): track 0.00 -> 73.2 mm
- net Net-(J17-Pad2): track 0.00 -> 67.0 mm
- net +5V: track 0.00 -> 65.1 mm
- net Net-(C24-Pad1): track 0.00 -> 57.5 mm, vias 0 -> 2
- net Net-(R17-Pad1): track 0.00 -> 49.8 mm, vias 0 -> 2
- net Net-(J7-Pad13): track 0.00 -> 48.6 mm
- net Net-(C14-Pad1): track 0.00 -> 47.5 mm
- net Net-(J11-Pad3): track 0.00 -> 44.6 mm, vias 0 -> 2
- net Net-(J11-Pad1): track 0.00 -> 44.5 mm
- net Net-(C19-Pad1): track 0.00 -> 42.4 mm
- net -5V: track 0.00 -> 41.2 mm
- net Net-(C20-Pad1): track 0.00 -> 40.3 mm
- net Net-(J6-Pad1): track 0.00 -> 40.1 mm
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- added copper zone on F.Cu, net (none)
- added copper zone on B.Cu, net GND
Other:
- board outline added: 110.6 x 83.2 mm
- net class Default: clearance 0.2 -> 0.1
- rule trace_clearance: 0.2 -> 0.1
