File: pcb/ASBF.kicad_pcb (KiCad board)
At the start: 2 copper layers, 110.6 x 83.2 mm, 75 parts, among them J1 Conn_01x02, J10 Conn_01x01, J11 Conn_01x03, J12 Conn_01x03, J13 Conn_01x03, J14 Conn_01x02, J15 Conn_01x03, J16 Conn_01x02, J17 Screw_Terminal_01x03, J2 Screw_Terminal_01x02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

Commit message: pcb v2.1
Parts:
- added C13: 1nf, Resistor_SMD:R_0805_2012Metric, B.Cu at (125.3, 74.5)
- added H3: MountingHole, MountingHole:MountingHole_2.5mm, F.Cu at (102.7, 43.8)
- added H4: MountingHole, MountingHole:MountingHole_2.5mm, F.Cu at (207.7, 121.3)
- R5: value 47 -> 2000
- moved R3 4.62 mm to (119.2, 84.4), turned to 0 degrees
- moved R1 3.30 mm to (115.2, 82.9)
- moved J2 2.72 mm to (114.7, 48.2)
- moved J3 2.53 mm to (132.5, 48.1)
- moved C9 2.42 mm to (112.6, 57.7)
- moved H1 0.70 mm to (102.7, 121.3)
- moved J1 0.50 mm to (109.5, 84.4)
- moved H2 0.36 mm to (207.7, 43.8)
- moved R5 0.13 mm to (122.7, 74.4)
Connections:
- R3 pad 2: Net-(R3-Pad2) -> Net-(C13-Pad2)
- R5 pad 1: Net-(R3-Pad2) -> Net-(C13-Pad2)
- U1 pad 3: Net-(R4-Pad2) -> Net-(C13-Pad2)
- U1 pad 4: Net-(R3-Pad2) -> Net-(R4-Pad2)
Routing:
- net GND: track 652.3 -> 689.9 mm
- net Net-(C13-Pad2): track 0.00 -> 16.9 mm
- net Net-(R3-Pad2): track 11.0 -> 0.00 mm
- net Net-(J1-Pad1): track 13.8 -> 8.30 mm
- net Net-(R4-Pad2): track 16.7 -> 21.0 mm, vias 0 -> 2
- net Net-(C1-Pad2): track 12.2 -> 15.1 mm
- net +3V3: track 277.1 -> 274.8 mm
- net -5V: track 41.2 -> 42.6 mm
- net +5V: track 65.1 -> 64.1 mm
- added copper zone on F.Cu, net GND
- removed copper zone on F.Cu, net (none)

Commit message: version 2.0
Parts:
- J11: Control: renamed from J11
- J12: 3v3: renamed from J12
- J13: GND: renamed from J13
- J14: A-B: renamed from J14
- J15:Ref. Gnd B: renamed from J15
- J16: Salida B DAC: renamed from J16
- J17: Tx Rx GND: renamed from J17
- J1: Antena In: renamed from J1
- J2: 3v3  GND: renamed from J2
- J3: GND -5v  +5v: renamed from J3
- J5: Ref. Gnd A: renamed from J5
- J6: Salida A DAC: renamed from J6
- J7: canal Auxiliar DAC: renamed from J7
- RV1: Ganancia: renamed from RV1
- RV2: Ref. 0V: renamed from RV2
- RV3: Vmax Conversion: renamed from RV3
- U2: ADC: renamed from U2
- U3: DAC: renamed from U3
- renumbered J4 to FPGA
Routing:
- net GND: track 689.9 -> 718.6 mm
Other:
- board text added: "Grilla utilizada: 0,1 mm Margen General: 0.5 mm Distancia al borde: 0.5mm Espesor de PCB: 1.6 mm Terminación Superficial: HASL Vía: 1.6/0.8 mm Pista en pad smd: 0.3 mm Pista en pad smd: 0.4 mm Pista en general: 0.8 mm"
- board text added: "Ind. Argentina"
- board text added: "Modelo: Adquisidor de senales V1.0 Fecha: 09/08/2021"

Commit message: correcciones agregadas
Parts:
- added FID1: Fiducial, Fiducial:Fiducial_1.5mm_Mask3mm, B.Cu at (103.0, 49.0)
- added FID2: Fiducial, Fiducial:Fiducial_1.5mm_Mask3mm, B.Cu at (108.0, 121.0)
- added FID3: Fiducial, Fiducial:Fiducial_1.5mm_Mask3mm, B.Cu at (208.0, 116.0)
- added FID4: Fiducial, Fiducial:Fiducial_1.5mm_Mask3mm, B.Cu at (203.0, 44.0)
- C1: value 0.33uf -> 0.33uF
- C10, C16, C17, C4, C9: value 10uf -> 10uF
- C11, C2, C3, C5, C7: value 0.1uf -> 0.1uF
- C12: value 1uf -> 1uF
- C14, C15, C18, C19, C20, C21, C22, C23, C24: value 100nf -> 100nF
- C6: value 10pf -> 10pF
- C8: value 0,1 uf -> 0,1 uF
- J10: test: renamed from J10
- J14: Out Dif.: renamed from J14: A-B
- J15: Ref. GND: renamed from J15:Ref. Gnd B
- J16: Out canal B DAC: renamed from J16: Salida B DAC
- J17: GND  RX  TX: renamed from J17: Tx Rx GND
- J1: Input : renamed from J1: Antena In
- J4: FPGA: renamed from FPGA
- J5: Ref. GND: renamed from J5: Ref. Gnd A
- J6: Out Canal A DAC: renamed from J6: Salida A DAC
- J7: DAC Canal B: renamed from J7: canal Auxiliar DAC
- J8: Bias B: renamed from J8
- J9: Bias A: renamed from J9
- RV1: Gan.: renamed from RV1: Ganancia
- RV2: Ref. 0V.: renamed from RV2: Ref. 0V
- RV3: Ref. Conv.: renamed from RV3: Vmax Conversion
- U2: renamed from U2: ADC
- U3: renamed from U3: DAC
- turned J14: Out Dif. to 90 degrees
Other:
- net class Default: clearance 0.1 -> 0.125
- rule trace_clearance: 0.1 -> 0.125
