File: pcb/DAC.sch (KiCad schematic (older format))
At the start: 40 parts, among them J10 Conn_01x01, J11 Conn_01x03, J12 Conn_01x03, J13 Conn_01x03, J14 Conn_01x02, J15 Conn_01x03, J16 Conn_01x02, J5 Conn_01x03, J6 Conn_01x02, J7 Conn_01x13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

Commit message: 1ra correcciones segun revision 1ra
Parts:
- C12, C16, C17: footprint Capacitor_THT:CP_Radial_D4.0mm_P1.50mm -> Resistor_SMD:R_0805_2012Metric
- C14, C15, C18, C19, C20, C21, C22, C23, C24: footprint Capacitor_THT:C_Disc_D3.0mm_W1.6mm_P2.50mm -> Resistor_SMD:R_0805_2012Metric
- R12, R13, R14, R15, R16, R17, R18, R19, R20, R21, R22: footprint Resistor_THT:R_Axial_DIN0207_L6.3mm_D2.5mm_P7.62mm_Horizontal -> Resistor_SMD:R_1206_3216Metric
Other:
- moved on the sheet: R17

Commit message: 1ra correcciones segun revision 1ra
Parts:
- added H1, H2: MountingHole, MountingHole:MountingHole_2.5mm, symbol Mechanical:MountingHole
Changed lines of the file:
@@
 	5400 4950 5400 5050
 Connection ~ 5400 4950
+$Comp
+L Mechanical:MountingHole H?
+U 1 1 60EF3943
+P 9100 6200
+AR Path="/60DC5AA5/60EF3943" Ref="H?"  Part="1"
+AR Path="/60E06463/60EF3943" Ref="H1"  Part="1"
+F 0 "H1" H 9200 6246 50  0000 L CNN
+F 1 "MountingHole" H 9200 6155 50  0000 L CNN
+F 2 "MountingHole:MountingHole_2.5mm" H 9100 6200 50  0001 C CNN
+F 3 "~" H 9100 6200 50  0001 C CNN
+	1    9100 6200
+	1    0    0    -1
+$EndComp
+$Comp
+L Mechanical:MountingHole H?
+U 1 1 60EF3949
+P 10100 6200
+AR Path="/60DC5AA5/60EF3949" Ref="H?"  Part="1"
+AR Path="/60E06463/60EF3949" Ref="H2"  Part="1"
+F 0 "H2" H 10200 6246 50  0000 L CNN
+F 1 "MountingHole" H 10200 6155 50  0000 L CNN
+F 2 "MountingHole:MountingHole_2.5mm" H 10100 6200 50  0001 C CNN
+F 3 "~" H 10100 6200 50  0001 C CNN
+	1    10100 6200
+	1    0    0    -1
+$EndComp
 $EndSCHEMATC

Commit message: Realizado de PCB
Parts:
- C12, C16, C17: footprint Resistor_SMD:R_0805_2012Metric -> Capacitor_THT:CP_Radial_D4.0mm_P1.50mm
- C21, C23: value 100NF -> 100nf
Changed lines of the file:
@@
 Sheet 2 4
 Title "Generacion de Seniales"
-Date "2021-07-05"
-Rev "V1.0"
+Date "2021-07-13"
+Rev "V1.1"
 Comp "Autor: Narvaez Pablo"
 Comment1 "Revision: 1ra"
@@
 F 0 "C12" H 6265 1796 50  0000 L CNN
 F 1 "1uf" H 6265 1705 50  0000 L CNN
-F 2 "Resistor_SMD:R_0805_2012Metric" H 6150 1750 50  0001 C CNN
+F 2 "Capacitor_THT:CP_Radial_D4.0mm_P1.50mm" H 6150 1750 50  0001 C CNN
 F 3 "~" H 6150 1750 50  0001 C CNN
 	1    6150 1750
@@
 P 8950 3750
 F 0 "C23" V 9202 3750 50  0000 C CNN
-F 1 "100NF" V 9111 3750 50  0000 C CNN
+F 1 "100nf" V 9111 3750 50  0000 C CNN
 F 2 "Resistor_SMD:R_0805_2012Metric" H 8988 3600 50  0001 C CNN
 F 3 "~" H 8950 3750 50  0001 C CNN
@@
 F 0 "C17" H 4565 1996 50  0000 L CNN
 F 1 "10uf" H 4565 1905 50  0000 L CNN
-F 2 "Resistor_SMD:R_0805_2012Metric" H 4450 1950 50  0001 C CNN
+F 2 "Capacitor_THT:CP_Radial_D4.0mm_P1.50mm" H 4450 1950 50  0001 C CNN
 F 3 "~" H 4450 1950 50  0001 C CNN
 	1    4450 1950
@@
 F 0 "C16" H 5815 1996 50  0000 L CNN
 F 1 "10uf" H 5815 1905 50  0000 L CNN
-F 2 "Resistor_SMD:R_0805_2012Metric" H 5700 1950 50  0001 C CNN
+F 2 "Capacitor_THT:CP_Radial_D4.0mm_P1.50mm" H 5700 1950 50  0001 C CNN
 F 3 "~" H 5700 1950 50  0001 C CNN
 	1    5700 1950
@@
 P 8100 3800
 F 0 "C21" V 8352 3800 50  0000 C CNN
-F 1 "100NF" V 8261 3800 50  0000 C CNN
+F 1 "100nf" V 8261 3800 50  0000 C CNN
 F 2 "Resistor_SMD:R_0805_2012Metric" H 8138 3650 50  0001 C CNN
 F 3 "~" H 8100 3800 50  0001 C CNN

Commit message: pcb v2.1
Parts:
- added H3, H4: MountingHole, MountingHole:MountingHole_2.5mm, symbol Mechanical:MountingHole
Changed lines of the file:
@@
 	5250 2200 5700 2200
 Wire Wire Line
-	5250 1650 5000 1650
+	5250 1650 5050 1650
 Connection ~ 5250 1650
 Wire Wire Line
@@
 Connection ~ 4450 1650
 Wire Wire Line
-	4450 1650 4800 1650
+	4450 1650 4750 1650
 Wire Wire Line
 	4200 1300 5200 1300
@@
 	1    0    0    -1
 $EndComp
+$Comp
+L power:PWR_FLAG #FLG0102
+U 1 1 6109EAD5
+P 4750 1650
+F 0 "#FLG0102" H 4750 1725 50  0001 C CNN
+F 1 "PWR_FLAG" H 4750 1823 50  0000 C CNN
+F 2 "" H 4750 1650 50  0001 C CNN
+F 3 "~" H 4750 1650 50  0001 C CNN
+	1    4750 1650
+	1    0    0    -1
+$EndComp
+Connection ~ 4750 1650
+Wire Wire Line
+	4750 1650 4800 1650
+$Comp
+L power:PWR_FLAG #FLG0103
+U 1 1 610A03E8
+P 5050 1650
+F 0 "#FLG0103" H 5050 1725 50  0001 C CNN
+F 1 "PWR_FLAG" H 5050 1823 50  0000 C CNN
+F 2 "" H 5050 1650 50  0001 C CNN
+F 3 "~" H 5050 1650 50  0001 C CNN
+	1    5050 1650
+	1    0    0    -1
+$EndComp
+Connection ~ 5050 1650
+Wire Wire Line
+	5050 1650 5000 1650
+$Comp
+L Mechanical:MountingHole H?
+U 1 1 610CB41D
+P 9100 5950
+AR Path="/60DC5AA5/610CB41D" Ref="H?"  Part="1"
+AR Path="/60E06463/610CB41D" Ref="H3"  Part="1"
+F 0 "H3" H 9200 5996 50  0000 L CNN
+F 1 "MountingHole" H 9200 5905 50  0000 L CNN
+F 2 "MountingHole:MountingHole_2.5mm" H 9100 5950 50  0001 C CNN
+F 3 "~" H 9100 5950 50  0001 C CNN
+	1    9100 5950
+	1    0    0    -1
+$EndComp
+$Comp
+L Mechanical:MountingHole H?
+U 1 1 610D69A5
+P 10100 5950
+AR Path="/60DC5AA5/610D69A5" Ref="H?"  Part="1"
+AR Path="/60E06463/610D69A5" Ref="H4"  Part="1"
+F 0 "H4" H 10200 5996 50  0000 L CNN
+F 1 "MountingHole" H 10200 5905 50  0000 L CNN
+F 2 "MountingHole:MountingHole_2.5mm" H 10100 5950 50  0001 C CNN
+F 3 "~" H 10100 5950 50  0001 C CNN
+	1    10100 5950
+	1    0    0    -1
+$EndComp
