File: pcb/ADC.sch (KiCad schematic (older format))
At the start: 31 parts, among them J1 Conn_01x02, J2 Screw_Terminal_01x02, J3 Screw_Terminal_01x03, U1 LMH6702MF, U2 ADC08060

Commit message: 1ra correcciones segun revision 1ra
Parts:
- C1, C11, C2, C3, C5, C6, C7, C8: footprint Capacitor_THT:C_Disc_D3.0mm_W1.6mm_P2.50mm -> Resistor_SMD:R_0805_2012Metric
- C10, C4, C9: footprint Capacitor_THT:CP_Radial_D4.0mm_P1.50mm -> Resistor_SMD:R_0805_2012Metric
- R1, R10, R11, R2, R3, R4, R5, R6, R7, R8, R9: footprint Resistor_THT:R_Axial_DIN0207_L6.3mm_D2.5mm_P7.62mm_Horizontal -> Resistor_SMD:R_1206_3216Metric
Other:
- moved on the sheet: J1
Changed lines of the file:
@@
 Date "2021-07-05"
 Rev "V1.0"
-Comp ""
-Comment1 ""
-Comment2 ""
-Comment3 ""
-Comment4 ""
+Comp "Autor: Narvaez Pablo"
+Comment1 "Revision: 1ra"
+Comment2 "Revisor Alumno: Ariel Cerfoglia"
+Comment3 "Revisor Docente: Diego Brengi"
+Comment4 "Licencia: GPLv3"
 $EndDescr
 Wire Wire Line
@@
 F 0 "C8" V 6702 2050 50  0000 C CNN
 F 1 "0,1 uf" V 6611 2050 50  0000 C CNN
-F 2 "Capacitor_THT:C_Disc_D3.0mm_W1.6mm_P2.50mm" H 6488 1900 50  0001 C CNN
+F 2 "Resistor_SMD:R_0805_2012Metric" H 6488 1900 50  0001 C CNN
 F 3 "~" H 6450 2050 50  0001 C CNN
 	1    6450 2050
@@
 F 0 "C9" H 6865 2096 50  0000 L CNN
 F 1 "10uf" H 6865 2005 50  0000 L CNN
-F 2 "Capacitor_THT:CP_Radial_D4.0mm_P1.50mm" H 6750 2050 50  0001 C CNN
+F 2 "Resistor_SMD:R_0805_2012Metric" H 6750 2050 50  0001 C CNN
 F 3 "~" H 6750 2050 50  0001 C CNN
 	1    6750 2050
@@
 F 0 "C6" H 6215 3296 50  0000 L CNN
 F 1 "10pf" H 6215 3205 50  0000 L CNN
-F 2 "Capacitor_THT:C_Disc_D3.0mm_W1.6mm_P2.50mm" H 6138 3100 50  0001 C CNN
+F 2 "Resistor_SMD:R_0805_2012Metric" H 6138 3100 50  0001 C CNN
 F 3 "~" H 6100 3250 50  0001 C CNN
 	1    6100 3250
@@
 F 0 "R6" V 2407 4200 50  0000 C CNN
 F 1 "4.7k" V 2316 4200 50  0000 C CNN
-F 2 "Resistor_THT:R_Axial_DIN0207_L6.3mm_D2.5mm_P7.62mm_Horizontal" V 2130 4200 50  0001 C CNN
+F 2 "Resistor_SMD:R_1206_3216Metric" V 2130 4200 50  0001 C CNN
 F 3 "~" H 2200 4200 50  0001 C CNN
 	1    2200 4200
@@
 F 0 "R5" H 2070 3446 50  0000 L CNN
 F 1 "47" H 2070 3355 50  0000 L CNN
-F 2 "Resistor_THT:R_Axial_DIN0207_L6.3mm_D2.5mm_P7.62mm_Horizontal" V 1930 3400 50  0001 C CNN
+F 2 "Resistor_SMD:R_1206_3216Metric" V 1930 3400 50  0001 C CNN
 F 3 "~" H 2000 3400 50  0001 C CNN
 	1    2000 3400
@@
 F 0 "R4" V 2707 2750 50  0000 C CNN
 F 1 "12" V 2616 2750 50  0000 C CNN
-F 2 "Resistor_THT:R_Axial_DIN0207_L6.3mm_D2.5mm_P7.62mm_Horizontal" V 2430 2750 50  0001 C CNN
+F 2 "Resistor_SMD:R_1206_3216Metric" V 2430 2750 50  0001 C CNN
 F 3 "~" H 2500 2750 50  0001 C CNN
 	1    2500 2750
@@
 F 0 "R2" V 2957 3750 50  0000 C CNN
 F 1 "1k" V 2866 3750 50  0000 C CNN
-F 2 "Resistor_THT:R_Axial_DIN0207_L6.3mm_D2.5mm_P7.62mm_Horizontal" V 2680 3750 50  0001 C CNN
+F 2 "Resistor_SMD:R_1206_3216Metric" V 2680 3750 50  0001 C CNN
 F 3 "~" H 2750 3750 50  0001 C CNN
 	1    2750 3750
@@
 F 0 "R1" H 1430 3354 50  0000 R CNN
 F 1 "100" H 1430 3445 50  0000 R CNN
-F 2 "Resistor_THT:R_Axial_DIN0207_L6.3mm_D2.5mm_P7.62mm_Horizontal" V 1430 3400 50  0001 C CNN
+F 2 "Resistor_SMD:R_1206_3216Metric" V 1430 3400 50  0001 C CNN
 F 3 "~" H 1500 3400 50  0001 C CNN
 	1    1500 3400
@@
 F 0 "R3" V 1957 3200 50  0000 C CNN
 F 1 "240" V 1866 3200 50  0000 C CNN
-F 2 "Resistor_THT:R_Axial_DIN0207_L6.3mm_D2.5mm_P7.62mm_Horizontal" V 1680 3200 50  0001 C CNN
+F 2 "Resistor_SMD:R_1206_3216Metric" V 1680 3200 50  0001 C CNN
 F 3 "~" H 1750 3200 50  0001 C CNN
 	1    1750 3200
@@
 F 0 "C2" V 3752 3800 50  0000 C CNN
 F 1 "0.1uf" V 3661 3800 50  0000 C CNN
-F 2 "Capacitor_THT:C_Disc_D3.0mm_W1.6mm_P2.50mm" H 3538 3650 50  0001 C CNN
+F 2 "Resistor_SMD:R_0805_2012Metric" H 3538 3650 50  0001 C CNN
 F 3 "~" H 3500 3800 50  0001 C CNN
 	1    3500 3800
@@
 F 0 "C1" V 2252 3800 50  0000 C CNN
 F 1 "0.33uf" V 2161 3800 50  0000 C CNN
-F 2 "Capacitor_THT:C_Disc_D3.0mm_W1.6mm_P2.50mm" H 2038 3650 50  0001 C CNN
+F 2 "Resistor_SMD:R_0805_2012Metric" H 2038 3650 50  0001 C CNN
 F 3 "~" H 2000 3800 50  0001 C CNN
 	1    2000 3800
@@
 F 0 "C3" V 4252 3800 50  0000 C CNN
 F 1 "0.1uf" V 4161 3800 50  0000 C CNN
-F 2 "Capacitor_THT:C_Disc_D3.0mm_W1.6mm_P2.50mm" H 4038 3650 50  0001 C CNN
+F 2 "Resistor_SMD:R_0805_2012Metric" H 4038 3650 50  0001 C CNN
 F 3 "~" H 4000 3800 50  0001 C CNN
 	1    4000 3800
@@
 L Connector_Generic:Conn_01x02 J1
 U 1 1 60DFD60D
-P 950 3550
-F 0 "J1" H 870 3225 50  0000 C CNN
-F 1 "Conn_01x02" H 870 3316 50  0000 C CNN
-F 2 "Connector_Coaxial:SMA_Amphenol_132134-16_Vertical" H 950 3550 50  0001 C CNN
-F 3 "~" H 950 3550 50  0001 C CNN
-	1    950  3550
+P 1050 3550
+F 0 "J1" H 1200 3650 50  0000 C CNN
+F 1 "Conn_01x02" H 1150 3750 50  0000 C CNN
+F 2 "Connector_Coaxial:SMA_Amphenol_132134-16_Vertical" H 1050 3550 50  0001 C CNN
+F 3 "~" H 1050 3550 50  0001 C CNN
+	1    1050 3550
 	-1   0    0    1
 $EndComp
@@
 F 0 "C7" H 6015 4546 50  0000 L CNN
 F 1 "0.1uf" H 6015 4455 50  0000 L CNN
-F 2 "Capacitor_THT:C_Disc_D3.0mm_W1.6mm_P2.50mm" H 5938 4350 50  0001 C CNN
+F 2 "Resistor_SMD:R_0805_2012Metric" H 5938 4350 50  0001 C CNN
 F 3 "~" H 5900 4500 50  0001 C CNN
 	1    5900 4500
@@
 F 0 "C5" H 5565 4446 50  0000 L CNN
 F 1 "0.1uf" H 5565 4355 50  0000 L CNN
-F 2 "Capacitor_THT:C_Disc_D3.0mm_W1.6mm_P2.50mm" H 5488 4250 50  0001 C CNN
+F 2 "Resistor_SMD:R_0805_2012Metric" H 5488 4250 50  0001 C CNN
 F 3 "~" H 5450 4400 50  0001 C CNN
 	1    5450 4400
@@
 F 0 "C4" H 5115 4446 50  0000 L CNN
 F 1 "10uf" H 5115 4355 50  0000 L CNN
-F 2 "Capacitor_THT:CP_Radial_D4.0mm_P1.50mm" H 5000 4400 50  0001 C CNN
+F 2 "Resistor_SMD:R_0805_2012Metric" H 5000 4400 50  0001 C CNN
 F 3 "~" H 5000 4400 50  0001 C CNN
 	1    5000 4400
@@
 F 0 "R10" H 6470 4546 50  0000 L CNN
 F 1 "1" H 6470 4455 50  0000 L CNN
-F 2 "Resistor_THT:R_Axial_DIN0207_L6.3mm_D2.5mm_P7.62mm_Horizontal" V 6330 4500 50  0001 C CNN
+F 2 "Resistor_SMD:R_1206_3216Metric" V 6330 4500 50  0001 C CNN
 F 3 "~" H 6400 4500 50  0001 C CNN
 	1    6400 4500
@@
 F 0 "R8" H 5220 2896 50  0000 L CNN
 F 1 "1" H 5220 2805 50  0000 L CNN
-F 2 "Resistor_THT:R_Axial_DIN0207_L6.3mm_D2.5mm_P7.62mm_Horizontal" V 5080 2850 50  0001 C CNN
+F 2 "Resistor_SMD:R_1206_3216Metric" V 5080 2850 50  0001 C CNN
 F 3 "~" H 5150 2850 50  0001 C CNN
 	1    5150 2850
@@
 U 1 1 6107421F
 P 2400 1300
-F 0 "J3" H 2318 975 50  0000 C CNN
-F 1 "Screw_Terminal_01x03" H 2318 1066 50  0000 C CNN
+F 0 "J3" H 2600 1450 50  0000 C CNN
+F 1 "Screw_Terminal_01x03" H 2650 1550 50  0000 C CNN
 F 2 "TerminalBlock:TerminalBlock_bornier-3_P5.08mm" H 2400 1300 50  0001 C CNN
 F 3 "~" H 2400 1300 50  0001 C CNN
@@
 U 1 1 60DFD607
 P 3150 3100
-F 0 "U1" H 3491 3146 50  0000 L CNN
-F 1 "LMH6702MF" H 3491 3055 50  0000 L CNN
+F 0 "U1" H 3250 2950 50  0000 L CNN
+F 1 "LMH6702MF" H 3150 2850 50  0000 L CNN
 F 2 "Package_TO_SOT_SMD:SOT-23-5" H 3150 3100 50  0001 L CNN
 F 3 "http://www.ti.com/lit/ds/symlink/lmh6702.pdf" H 3150 3100 50  0001 C CNN
@@
 F 0 "R7" V 3507 2750 50  0000 C CNN
 F 1 "200" V 3416 2750 50  0000 C CNN
-F 2 "Resistor_THT:R_Axial_DIN0207_L6.3mm_D2.5mm_P7.62mm_Horizontal" V 3230 2750 50  0001 C CNN
+F 2 "Resistor_SMD:R_1206_3216Metric" V 3230 2750 50  0001 C CNN
 F 3 "~" H 3300 2750 50  0001 C CNN
 	1    3300 2750
@@
 L power:GND #PWR0105
 U 1 1 60F878B4
-P 1150 4250
-F 0 "#PWR0105" H 1150 4000 50  0001 C CNN
-F 1 "GND" H 1155 4077 50  0000 C CNN
-F 2 "" H 1150 4250 50  0001 C CNN
-F 3 "" H 1150 4250 50  0001 C CNN
-	1    1150 4250
+P 1500 4250
+F 0 "#PWR0105" H 1500 4000 50  0001 C CNN
+F 1 "GND" H 1505 4077 50  0000 C CNN
+F 2 "" H 1500 4250 50  0001 C CNN
+F 3 "" H 1500 4250 50  0001 C CNN
+	1    1500 4250
 	1    0    0    -1
 $EndComp
@@
 F 0 "R11" H 8170 4246 50  0000 L CNN
 F 1 "4.7k" H 8170 4155 50  0000 L CNN
-F 2 "Resistor_THT:R_Axial_DIN0207_L6.3mm_D2.5mm_P7.62mm_Horizontal" V 8030 4200 50  0001 C CNN
+F 2 "Resistor_SMD:R_1206_3216Metric" V 8030 4200 50  0001 C CNN
 F 3 "~" H 8100 4200 50  0001 C CNN
 	1    8100 4200
@@
 F 0 "R9" V 6057 3100 50  0000 C CNN
 F 1 "22" V 5966 3100 50  0000 C CNN
-F 2 "Resistor_THT:R_Axial_DIN0207_L6.3mm_D2.5mm_P7.62mm_Horizontal" V 5780 3100 50  0001 C CNN
+F 2 "Resistor_SMD:R_1206_3216Metric" V 5780 3100 50  0001 C CNN
 F 3 "~" H 5850 3100 50  0001 C CNN
 	1    5850 3100
@@
 	1500 3200 1500 3250
 Wire Wire Line
-	1150 3450 1150 3200
-Wire Wire Line
-	1150 3200 1500 3200
+	1250 3450 1250 3200
 Wire Wire Line
 	2750 3600 2750 3550
@@
 	2000 3950 1500 3950
 Wire Wire Line
-	1150 3550 1150 3950
-Connection ~ 1150 3950
-Wire Wire Line
-	1150 3950 1150 4250
+	1500 3950 1500 4250
 Wire Wire Line
 	1500 3550 1500 3950
@@
 	1700 2750 1300 2750
 Connection ~ 1700 2750
-Wire Wire Line
-	1150 3950 1500 3950
 $Comp
 L power:GND #PWR0123
@@
 	1300 2900 1300 2750
 Wire Notes Line
-	800  2000 4400 2000
-Wire Notes Line
 	4400 2000 4400 4750
 Wire Notes Line
-	4400 4750 800  4750
-Wire Notes Line
-	800  4750 800  2000
+	700  4750 700  2000
 Text Notes 900  4700 0    50   ~ 10
 Adecuacion de senial
@@
 U 1 1 60DFD6C8
 P 7200 3550
-F 0 "U2" H 7200 4528 50  0000 C CNN
-F 1 "ADC08060" H 7200 4437 50  0000 C CNN
+F 0 "U2" H 6400 4400 50  0000 L CNN
+F 1 "ADC08060" H 6450 4300 50  0000 C CNN
 F 2 "Package_SO:TSSOP-24_4.4x7.8mm_P0.65mm" H 7200 3550 50  0001 C CNN
 F 3 "http://www.ti.com/lit/ds/symlink/adc08060.pdf" H 7200 3550 50  0001 C CNN
@@
 F 0 "C10" V 7698 2100 50  0000 C CNN
 F 1 "10uf" V 7789 2100 50  0000 C CNN
-F 2 "Capacitor_THT:CP_Radial_D4.0mm_P1.50mm" H 7950 2100 50  0001 C CNN
+F 2 "Resistor_SMD:R_0805_2012Metric" H 7950 2100 50  0001 C CNN
 F 3 "~" H 7950 2100 50  0001 C CNN
 	1    7950 2100
@@
 F 0 "C11" V 7752 2100 50  0000 C CNN
 F 1 "0.1uf" V 7661 2100 50  0000 C CNN
-F 2 "Capacitor_THT:C_Disc_D3.0mm_W1.6mm_P2.50mm" H 7538 1950 50  0001 C CNN
+F 2 "Resistor_SMD:R_0805_2012Metric" H 7538 1950 50  0001 C CNN
 F 3 "~" H 7500 2100 50  0001 C CNN
 	1    7500 2100
@@
 Wire Wire Line
 	1900 1000 1900 1200
+Wire Notes Line
+	700  2000 4400 2000
+Wire Notes Line
+	700  4750 4400 4750
+Wire Wire Line
+	1250 3550 1250 3950
+Wire Wire Line
+	1250 3200 1500 3200
+Wire Wire Line
+	1250 3950 1500 3950
 $EndSCHEMATC

Commit message: 1ra correcciones segun revision 1ra
Changed lines of the file:
@@
 	3050 4350 3050 4500
 Wire Notes Line
-	8400 1050 8400 5000
-Wire Notes Line
-	8400 5000 4850 5000
-Wire Notes Line
-	4850 5000 4850 1050
+	8400 5200 4850 5200
 Wire Notes Line
 	4850 1050 8400 1050
@@
 Wire Wire Line
 	1250 3950 1500 3950
+Wire Notes Line
+	4850 5200 4850 1050
+Wire Notes Line
+	8400 5200 8400 1050
 $EndSCHEMATC

Commit message: Realizado de PCB
Parts:
- removed U2: ADC08060, Package_SO:TSSOP-24_4.4x7.8mm_P0.65mm, symbol Analog_ADC:ADC08060
- added U2: ADC080200, Package_SO:TSSOP-24_4.4x7.8mm_P0.65mm, symbol ASBF-rescue:ADC080200-adc080200
- C10, C4, C9: footprint Resistor_SMD:R_0805_2012Metric -> Capacitor_THT:CP_Radial_D4.0mm_P1.50mm
Changed lines of the file:
@@
 $Descr A4 11693 8268
 encoding utf-8
-Sheet 4 4
+Sheet 3 4
 Title "Adquisicion de datos"
 Date "2021-07-05"
@@
 $EndDescr
 Wire Wire Line
-	6900 4350 7000 4350
-Connection ~ 7000 4350
-Wire Wire Line
 	6300 3400 6300 3350
 Wire Wire Line
@@
 F 0 "C9" H 6865 2096 50  0000 L CNN
 F 1 "10uf" H 6865 2005 50  0000 L CNN
-F 2 "Resistor_SMD:R_0805_2012Metric" H 6750 2050 50  0001 C CNN
+F 2 "Capacitor_THT:CP_Radial_D4.0mm_P1.50mm" H 6750 2050 50  0001 C CNN
 F 3 "~" H 6750 2050 50  0001 C CNN
 	1    6750 2050
@@
 F 3 "~" H 2500 4050 50  0001 C CNN
 	1    2500 4050
-	0    -1   -1   0
+	0    1    -1   0
 $EndComp
 $Comp
@@
 L Connector_Generic:Conn_01x02 J1
 U 1 1 60DFD60D
-P 1050 3550
-F 0 "J1" H 1200 3650 50  0000 C CNN
-F 1 "Conn_01x02" H 1150 3750 50  0000 C CNN
-F 2 "Connector_Coaxial:SMA_Amphenol_132134-16_Vertical" H 1050 3550 50  0001 C CNN
-F 3 "~" H 1050 3550 50  0001 C CNN
-	1    1050 3550
-	-1   0    0    1
+P 1050 3450
+F 0 "J1" H 1200 3550 50  0000 C CNN
+F 1 "Conn_01x02" H 1150 3650 50  0000 C CNN
+F 2 "Connector_Coaxial:SMA_Amphenol_132134-16_Vertical" H 1050 3450 50  0001 C CNN
+F 3 "~" H 1050 3450 50  0001 C CNN
+	1    1050 3450
+	-1   0    0    -1
 $EndComp
 Wire Wire Line
@@
 $EndComp
 Wire Wire Line
-	2600 1200 2800 1200
-Wire Wire Line
 	2600 1400 2650 1400
 $Comp
@@
 F 0 "C4" H 5115 4446 50  0000 L CNN
 F 1 "10uf" H 5115 4355 50  0000 L CNN
-F 2 "Resistor_SMD:R_0805_2012Metric" H 5000 4400 50  0001 C CNN
+F 2 "Capacitor_THT:CP_Radial_D4.0mm_P1.50mm" H 5000 4400 50  0001 C CNN
 F 3 "~" H 5000 4400 50  0001 C CNN
 	1    5000 4400
@@
 Text HLabel 8700 3950 2    50   Input ~ 0
 CLK
-$Comp
-L Connector:Screw_Terminal_01x03 J3
-U 1 1 6107421F
-P 2400 1300
-F 0 "J3" H 2600 1450 50  0000 C CNN
-F 1 "Screw_Terminal_01x03" H 2650 1550 50  0000 C CNN
-F 2 "TerminalBlock:TerminalBlock_bornier-3_P5.08mm" H 2400 1300 50  0001 C CNN
-F 3 "~" H 2400 1300 50  0001 C CNN
-	1    2400 1300
-	-1   0    0    1
-$EndComp
 Wire Wire Line
 	1450 1200 1900 1200
@@
 $EndComp
 Wire Wire Line
-	2600 1300 3000 1300
-Wire Wire Line
 	2750 2750 3150 2750
 $Comp
@@
 U 1 1 610765E7
 P 1250 1300
-F 0 "J2" H 1168 975 50  0000 C CNN
-F 1 "Screw_Terminal_01x02" H 1168 1066 50  0000 C CNN
+F 0 "J2" H 1350 1600 50  0000 C CNN
+F 1 "Screw_Terminal_01x02" H 1200 1450 50  0000 C CNN
 F 2 "TerminalBlock:TerminalBlock_bornier-2_P5.08mm" H 1250 1300 50  0001 C CNN
 F 3 "~" H 1250 1300 50  0001 C CNN
@@
 	6750 2300 6750 2250
 Wire Wire Line
-	7100 2750 7000 2750
-Connection ~ 7000 2750
-Connection ~ 7100 2750
-Wire Wire Line
-	7100 4350 7050 4350
-Wire Wire Line
-	7100 4350 7300 4350
-Connection ~ 7100 4350
-Wire Wire Line
-	6900 2750 7000 2750
-$Comp
-L Analog_ADC:ADC08060 U2
-U 1 1 60DFD6C8
-P 7200 3550
-F 0 "U2" H 6400 4400 50  0000 L CNN
-F 1 "ADC08060" H 6450 4300 50  0000 C CNN
-F 2 "Package_SO:TSSOP-24_4.4x7.8mm_P0.65mm" H 7200 3550 50  0001 C CNN
-F 3 "http://www.ti.com/lit/ds/symlink/adc08060.pdf" H 7200 3550 50  0001 C CNN
-	1    7200 3550
-	1    0    0    -1
-$EndComp
-Wire Wire Line
 	6450 2200 6450 2250
 Wire Wire Line
@@
 F 0 "C10" V 7698 2100 50  0000 C CNN
 F 1 "10uf" V 7789 2100 50  0000 C CNN
-F 2 "Resistor_SMD:R_0805_2012Metric" H 7950 2100 50  0001 C CNN
+F 2 "Capacitor_THT:CP_Radial_D4.0mm_P1.50mm" H 7950 2100 50  0001 C CNN
 F 3 "~" H 7950 2100 50  0001 C CNN
 	1    7950 2100
@@
 Connection ~ 7050 4350
 Wire Wire Line
-	7050 4350 7000 4350
-Wire Wire Line
 	7400 4350 7400 4750
 Wire Wire Line
@@
 Wire Notes Line
 	8400 5200 8400 1050
+Wire Wire Line
+	7050 4350 7100 4350
+$Comp
+L ASBF-rescue:ADC080200-adc080200 U2
+U 1 1 60F9C145
+P 7200 3550
+AR Path="/60F9C145" Ref="U2"  Part="1"
+AR Path="/60DC5AA5/60F9C145" Ref="U2"  Part="1"
+F 0 "U2" H 7200 4531 50  0000 C CNN
+F 1 "ADC080200" H 7200 4440 50  0000 C CNN
+F 2 "Package_SO:TSSOP-24_4.4x7.8mm_P0.65mm" H 7200 3550 50  0001 C CNN
+F 3 "http://www.ti.com/lit/ds/symlink/adc080200.pdf" H 7200 3550 50  0001 C CNN
+	1    7200 3550
+	1    0    0    -1
+$EndComp
+Wire Wire Line
+	7000 2750 7100 2750
+Connection ~ 7100 2750
+Wire Wire Line
+	7000 4350 7050 4350
+Wire Wire Line
+	6900 4350 7000 4350
+Connection ~ 7000 4350
+Wire Wire Line
+	6900 2750 7000 2750
+Connection ~ 7000 2750
+Wire Wire Line
+	7300 4350 7400 4350
+Connection ~ 7400 4350
+$Comp
+L Connector:Screw_Terminal_01x03 J3
+U 1 1 6107421F
+P 2400 1300
+F 0 "J3" H 2600 1450 50  0000 C CNN
+F 1 "Screw_Terminal_01x03" H 2650 1550 50  0000 C CNN
+F 2 "TerminalBlock:TerminalBlock_bornier-3_P5.08mm" H 2400 1300 50  0001 C CNN
+F 3 "~" H 2400 1300 50  0001 C CNN
+	1    2400 1300
+	-1   0    0    -1
+$EndComp
+Wire Wire Line
+	3000 1300 2600 1300
+Wire Wire Line
+	2800 1200 2600 1200
 $EndSCHEMATC

Commit message: pcb v2.1
Parts:
- added C13: 1nf, Resistor_SMD:R_0805_2012Metric, symbol Device:C
- R5: value 47 -> 2000
Connections:
- net at R3.2, R5.1: now also U1.3 (+), C13.2; no longer U1.4 (-)
- net at C1.2, R5.2, RV2.2: now also C13.1
- net at R4.2, R7.1: now also U1.4 (-); no longer U1.3 (+)
Other:
- moved on the sheet: R2
Changed lines of the file:
@@
 P 2000 3400
 F 0 "R5" H 2070 3446 50  0000 L CNN
-F 1 "47" H 2070 3355 50  0000 L CNN
+F 1 "2000" H 2070 3355 50  0000 L CNN
 F 2 "Resistor_SMD:R_1206_3216Metric" V 1930 3400 50  0001 C CNN
 F 3 "~" H 2000 3400 50  0001 C CNN
@@
 L Device:R R2
 U 1 1 60DFD574
-P 2750 3750
-F 0 "R2" V 2957 3750 50  0000 C CNN
-F 1 "1k" V 2866 3750 50  0000 C CNN
-F 2 "Resistor_SMD:R_1206_3216Metric" V 2680 3750 50  0001 C CNN
-F 3 "~" H 2750 3750 50  0001 C CNN
-	1    2750 3750
+P 2850 3850
+F 0 "R2" V 3057 3850 50  0000 C CNN
+F 1 "1k" V 2966 3850 50  0000 C CNN
+F 2 "Resistor_SMD:R_1206_3216Metric" V 2780 3850 50  0001 C CNN
+F 3 "~" H 2850 3850 50  0001 C CNN
+	1    2850 3850
 	-1   0    0    1
 $EndComp
@@
 $EndComp
 $Comp
-L Device:R_POT RV2
-U 1 1 60DFD586
-P 2500 4050
-F 0 "RV2" V 2386 4050 50  0000 C CNN
-F 1 "1k" V 2295 4050 50  0000 C CNN
-F 2 "Potentiometer_THT:Potentiometer_Bourns_3266Y_Vertical" H 2500 4050 50  0001 C CNN
-F 3 "~" H 2500 4050 50  0001 C CNN
-	1    2500 4050
-	0    1    -1   0
-$EndComp
-$Comp
 L Device:R_POT RV1
 U 1 1 60DFD58C
@@
 L power:+3.3V #PWR0112
 U 1 1 60DFD5E0
-P 2750 3550
-F 0 "#PWR0112" H 2750 3400 50  0001 C CNN
-F 1 "+3.3V" H 2765 3723 50  0000 C CNN
-F 2 "" H 2750 3550 50  0001 C CNN
-F 3 "" H 2750 3550 50  0001 C CNN
-	1    2750 3550
+P 2850 3650
+F 0 "#PWR0112" H 2850 3500 50  0001 C CNN
+F 1 "+3.3V" H 2865 3823 50  0000 C CNN
+F 2 "" H 2850 3650 50  0001 C CNN
+F 3 "" H 2850 3650 50  0001 C CNN
+	1    2850 3650
 	1    0    0    -1
 $EndComp
@@
 Wire Wire Line
 	3450 3100 3550 3100
-Wire Wire Line
-	2750 2750 2750 3000
-Wire Wire Line
-	2750 3000 2850 3000
 $Comp
 L Connector_Generic:Conn_01x02 J1
@@
 CLK
 Wire Wire Line
-	1450 1200 1900 1200
+	1450 1200 1650 1200
 Wire Wire Line
 	1450 1300 1500 1300
@@
 	1    0    0    -1
 $EndComp
-Wire Wire Line
-	2750 2750 3150 2750
 $Comp
 L Connector:Screw_Terminal_01x02 J2
@@
 Wire Wire Line
 	4000 4250 4000 3950
-Connection ~ 2750 2750
-Wire Wire Line
-	2650 2750 2750 2750
 Wire Wire Line
 	2350 2750 2200 2750
@@
 	1250 3450 1250 3200
 Wire Wire Line
-	2750 3600 2750 3550
-Wire Wire Line
-	2750 3900 2750 4050
-Wire Wire Line
-	2750 4050 2650 4050
+	2850 3700 2850 3650
 Wire Wire Line
 	2350 4050 2200 4050
@@
 	2500 3550 2500 3900
 Wire Wire Line
-	2850 3200 2000 3200
-Wire Wire Line
 	2000 3250 2000 3200
 Wire Wire Line
@@
 Connection ~ 1500 3950
 Wire Wire Line
-	2000 3550 2500 3550
+	2000 3550 2400 3550
 Connection ~ 2000 3550
 Wire Wire Line
 	1900 3200 2000 3200
-Connection ~ 2000 3200
 Wire Wire Line
 	1600 3200 1500 3200
@@
 $EndComp
 Wire Wire Line
-	3000 1300 2600 1300
-Wire Wire Line
-	2800 1200 2600 1200
+	3000 1300 2900 1300
+Wire Wire Line
+	2800 1200 2700 1200
+Wire Wire Line
+	2650 2750 2700 2750
+Wire Wire Line
+	2850 3200 2700 3200
+Wire Wire Line
+	2700 3200 2700 2750
+Connection ~ 2700 2750
+Wire Wire Line
+	2700 2750 3150 2750
+Wire Wire Line
+	2850 3000 2350 3000
+Wire Wire Line
+	2350 3000 2350 3200
+Wire Wire Line
+	2350 3200 2000 3200
+Connection ~ 2000 3200
+$Comp
+L Device:C C13
+U 1 1 61067490
+P 2400 3400
+F 0 "C13" V 2250 3400 50  0000 C CNN
+F 1 "1nf" V 2150 3400 50  0000 C CNN
+F 2 "Resistor_SMD:R_0805_2012Metric" H 2438 3250 50  0001 C CNN
+F 3 "~" H 2400 3400 50  0001 C CNN
+	1    2400 3400
+	-1   0    0    1
+$EndComp
+Connection ~ 2400 3550
+Wire Wire Line
+	2400 3550 2500 3550
+Wire Wire Line
+	2400 3250 2400 3200
+Wire Wire Line
+	2400 3200 2350 3200
+Connection ~ 2350 3200
+$Comp
+L Device:R_POT RV2
+U 1 1 60DFD586
+P 2500 4050
+F 0 "RV2" V 2386 4050 50  0000 C CNN
+F 1 "1k" V 2295 4050 50  0000 C CNN
+F 2 "Potentiometer_THT:Potentiometer_Bourns_3266Y_Vertical" H 2500 4050 50  0001 C CNN
+F 3 "~" H 2500 4050 50  0001 C CNN
+	1    2500 4050
+	0    1    -1   0
+$EndComp
+Wire Wire Line
+	2850 4000 2850 4050
+Wire Wire Line
+	2650 4050 2850 4050
+$Comp
+L power:PWR_FLAG #FLG0101
+U 1 1 6108E2EC
+P 1650 1200
+F 0 "#FLG0101" H 1650 1275 50  0001 C CNN
+F 1 "PWR_FLAG" H 1650 1373 50  0000 C CNN
+F 2 "" H 1650 1200 50  0001 C CNN
+F 3 "~" H 1650 1200 50  0001 C CNN
+	1    1650 1200
+	1    0    0    -1
+$EndComp
+Connection ~ 1650 1200
+Wire Wire Line
+	1650 1200 1900 1200
+$Comp
+L power:PWR_FLAG #FLG0104
+U 1 1 610A2BCE
+P 1500 1300
+F 0 "#FLG0104" H 1500 1375 50  0001 C CNN
+F 1 "PWR_FLAG" V 1500 1428 50  0000 L CNN
+F 2 "" H 1500 1300 50  0001 C CNN
+F 3 "~" H 1500 1300 50  0001 C CNN
+	1    1500 1300
+	0    1    1    0
+$EndComp
+Connection ~ 1500 1300
+$Comp
+L power:PWR_FLAG #FLG0105
+U 1 1 610A3B12
+P 2900 1300
+F 0 "#FLG0105" H 2900 1375 50  0001 C CNN
+F 1 "PWR_FLAG" H 2900 1473 50  0000 C CNN
+F 2 "" H 2900 1300 50  0001 C CNN
+F 3 "~" H 2900 1300 50  0001 C CNN
+	1    2900 1300
+	1    0    0    -1
+$EndComp
+Connection ~ 2900 1300
+Wire Wire Line
+	2900 1300 2600 1300
+$Comp
+L power:PWR_FLAG #FLG0106
+U 1 1 610A48F2
+P 2700 1200
+F 0 "#FLG0106" H 2700 1275 50  0001 C CNN
+F 1 "PWR_FLAG" H 2700 1373 50  0000 C CNN
+F 2 "" H 2700 1200 50  0001 C CNN
+F 3 "~" H 2700 1200 50  0001 C CNN
+	1    2700 1200
+	1    0    0    -1
+$EndComp
+Connection ~ 2700 1200
+Wire Wire Line
+	2700 1200 2600 1200
+$Comp
+L power:PWR_FLAG #FLG0107
+U 1 1 610A5C63
+P 7300 1850
+F 0 "#FLG0107" H 7300 1925 50  0001 C CNN
+F 1 "PWR_FLAG" H 7300 2023 50  0000 C CNN
+F 2 "" H 7300 1850 50  0001 C CNN
+F 3 "~" H 7300 1850 50  0001 C CNN
+	1    7300 1850
+	1    0    0    -1
+$EndComp
+Connection ~ 7300 1850
 $EndSCHEMATC

Commit message: correcciones agregadas
Parts:
- C1: value 0.33uf -> 0.33uF
- C10, C4, C9: value 10uf -> 10uF
- C11, C2, C3, C5, C7: value 0.1uf -> 0.1uF
- C6: value 10pf -> 10pF
- C8: value 0,1 uf -> 0,1 uF
Other:
- moved on the sheet: L1, R1, R11, R9
