File: pcb/ASBF.sch (KiCad schematic (older format))
At the start: 0 parts

Commit message: Realizado de PCB
Connections:
- no-connect marks 23 -> 21

Commit message: correcciones agregadas
Changed lines of the file:
@@
 F11 "CLK" I R 4350 2800 50
 $EndSheet
-$Comp
-L power:+5V #PWR?
-U 1 1 61049E41
-P 6250 2350
-AR Path="/60DC5AA5/61049E41" Ref="#PWR?"  Part="1"
-AR Path="/61049E41" Ref="#PWR0131"  Part="1"
-F 0 "#PWR0131" H 6250 2200 50  0001 C CNN
-F 1 "+5V" H 6265 2523 50  0000 C CNN
-F 2 "" H 6250 2350 50  0001 C CNN
-F 3 "" H 6250 2350 50  0001 C CNN
-	1    6250 2350
-	1    0    0    -1
-$EndComp
-Wire Wire Line
-	6100 2600 6250 2600
-Wire Wire Line
-	6250 2600 6250 2350
-Wire Wire Line
-	5450 2600 5250 2600
-Wire Wire Line
-	5250 2600 5250 2400
-$Comp
-L power:GND #PWR?
-U 1 1 610A0DAC
-P 5250 2400
-AR Path="/60DC5AA5/610A0DAC" Ref="#PWR?"  Part="1"
-AR Path="/610A0DAC" Ref="#PWR0139"  Part="1"
-F 0 "#PWR0139" H 5250 2150 50  0001 C CNN
-F 1 "GND" H 5255 2227 50  0000 C CNN
-F 2 "" H 5250 2400 50  0001 C CNN
-F 3 "" H 5250 2400 50  0001 C CNN
-	1    5250 2400
-	-1   0    0    1
-$EndComp
 NoConn ~ 6100 2700
 NoConn ~ 6100 2800
@@
 F0 "FPGA_Conector" 50
 F1 "FPGAConector.sch" 50
-F2 "VCC" I R 6100 2600 50
-F3 "N1" B R 6100 4600 50
-F4 "M2" B R 6100 4500 50
-F5 "P3" I R 6100 4400 50
-F6 "N3" B R 6100 4300 50
-F7 "M1" B R 6100 4200 50
-F8 "H2" B R 6100 4100 50
-F9 "G3" B R 6100 4000 50
-F10 "L2" B R 6100 3900 50
-F11 "L1" B R 6100 3800 50
-F12 "K2" B R 6100 3700 50
-F13 "J1" B R 6100 3600 50
-F14 "J3" B R 6100 3500 50
-F15 "A14" B R 6100 3400 50
-F16 "B15" B R 6100 3300 50
-F17 "A15" B R 6100 3200 50
-F18 "H1" B R 6100 3100 50
-F19 "C15" B R 6100 3000 50
-F20 "K3" B R 6100 2900 50
-F21 "A16" B R 6100 2800 50
-F22 "L3" B R 6100 2700 50
-F23 "M3" B R 6100 4700 50
-F24 "GND" I L 5450 2600 50
-F25 "R3" B L 5450 4900 50
-F26 "T3" B L 5450 4800 50
-F27 "R2" B L 5450 4700 50
-F28 "T1" B L 5450 4600 50
-F29 "T2" B L 5450 4500 50
-F30 "U1" B L 5450 4400 50
-F31 "W2" B L 5450 4300 50
-F32 "V2" B L 5450 4200 50
-F33 "W3" B L 5450 4100 50
-F34 "V3" B L 5450 4000 50
-F35 "W5" B L 5450 3900 50
-F36 "V4" B L 5450 3800 50
-F37 "U4" B L 5450 3700 50
-F38 "V5" B L 5450 3600 50
-F39 "W4" B L 5450 3500 50
-F40 "U5" B L 5450 3400 50
-F41 "U2" B L 5450 3300 50
-F42 "W6" B L 5450 3200 50
-F43 "U3" B L 5450 3100 50
-F44 "U7" B L 5450 3000 50
-F45 "W7" B L 5450 2900 50
-F46 "U8" B L 5450 2800 50
-F47 "V8" B L 5450 2700 50
+F2 "N1" B R 6100 4600 50
+F3 "M2" B R 6100 4500 50
+F4 "P3" I R 6100 4400 50
+F5 "N3" B R 6100 4300 50
+F6 "M1" B R 6100 4200 50
+F7 "H2" B R 6100 4100 50
+F8 "G3" B R 6100 4000 50
+F9 "L2" B R 6100 3900 50
+F10 "L1" B R 6100 3800 50
+F11 "K2" B R 6100 3700 50
+F12 "J1" B R 6100 3600 50
+F13 "J3" B R 6100 3500 50
+F14 "A14" B R 6100 3400 50
+F15 "B15" B R 6100 3300 50
+F16 "A15" B R 6100 3200 50
+F17 "H1" B R 6100 3100 50
+F18 "C15" B R 6100 3000 50
+F19 "K3" B R 6100 2900 50
+F20 "A16" B R 6100 2800 50
+F21 "L3" B R 6100 2700 50
+F22 "M3" B R 6100 4700 50
+F23 "GND" I L 5450 2600 50
+F24 "R3" B L 5450 4900 50
+F25 "T3" B L 5450 4800 50
+F26 "R2" B L 5450 4700 50
+F27 "T1" B L 5450 4600 50
+F28 "T2" B L 5450 4500 50
+F29 "U1" B L 5450 4400 50
+F30 "W2" B L 5450 4300 50
+F31 "V2" B L 5450 4200 50
+F32 "W3" B L 5450 4100 50
+F33 "V3" B L 5450 4000 50
+F34 "W5" B L 5450 3900 50
+F35 "V4" B L 5450 3800 50
+F36 "U4" B L 5450 3700 50
+F37 "V5" B L 5450 3600 50
+F38 "W4" B L 5450 3500 50
+F39 "U5" B L 5450 3400 50
+F40 "U2" B L 5450 3300 50
+F41 "W6" B L 5450 3200 50
+F42 "U3" B L 5450 3100 50
+F43 "U7" B L 5450 3000 50
+F44 "W7" B L 5450 2900 50
+F45 "U8" B L 5450 2800 50
+F46 "V8" B L 5450 2700 50
+F47 "VCC" I R 6100 2600 50
 $EndSheet
 NoConn ~ 5450 4900
