File: pcb/FPGAConector.sch (KiCad schematic (older format))
At the start: 1 part, among them J4 Conn_02x24_Counter_Clockwise

Commit message: Realizado de PCB
Parts:
- added J17: Screw_Terminal_01x03, TerminalBlock:TerminalBlock_bornier-3_P5.08mm, symbol Connector:Screw_Terminal_01x03
Connections:
- net GND: now also J17.3 (Pin_3)
- net N2: no longer names the net of J4.46 (Pin_46)
- net N2: now also J17.2 (Pin_2)
- net P1: no longer names the net of J4.47 (Pin_47)
- net P1: now also J17.1 (Pin_1)
Changed lines of the file:
@@
 $Descr A4 11693 8268
 encoding utf-8
-Sheet 3 4
+Sheet 4 4
 Title ""
 Date ""
@@
 Text HLabel 5950 2400 2    50   Input ~ 0
 VCC
-Text HLabel 5950 2500 2    50   BiDi ~ 0
-P1
-Text HLabel 5950 2600 2    50   BiDi ~ 0
-N2
 Text HLabel 5950 2700 2    50   BiDi ~ 0
 N1
@@
 V8
 Wire Notes Line
-	4700 2000 6550 2000
-Wire Notes Line
-	6550 2000 6550 4950
-Wire Notes Line
 	4700 4950 4700 2000
-Wire Notes Line
-	4700 4950 6550 4950
 Text Notes 4750 4850 0    50   ~ 10
 Conector FPGA
+$Comp
+L power:GND #PWR?
+U 1 1 60FCBB33
+P 6350 2800
+AR Path="/60DC5AA5/60FCBB33" Ref="#PWR?"  Part="1"
+AR Path="/60FCBB33" Ref="#PWR?"  Part="1"
+AR Path="/6101F213/60FCBB33" Ref="#PWR05"  Part="1"
+F 0 "#PWR05" H 6350 2550 50  0001 C CNN
+F 1 "GND" H 6355 2627 50  0000 C CNN
+F 2 "" H 6350 2800 50  0001 C CNN
+F 3 "" H 6350 2800 50  0001 C CNN
+	1    6350 2800
+	1    0    0    -1
+$EndComp
+Wire Notes Line
+	4700 2000 7950 2000
+Wire Notes Line
+	7950 4950 7950 2000
+Wire Notes Line
+	4700 4950 7950 4950
+$Comp
+L Connector:Screw_Terminal_01x03 J17
+U 1 1 60FC9BE6
+P 6650 2600
+F 0 "J17" H 6730 2642 50  0000 L CNN
+F 1 "Screw_Terminal_01x03" H 6730 2551 50  0000 L CNN
+F 2 "TerminalBlock:TerminalBlock_bornier-3_P5.08mm" H 6650 2600 50  0001 C CNN
+F 3 "~" H 6650 2600 50  0001 C CNN
+	1    6650 2600
+	1    0    0    -1
+$EndComp
+Wire Wire Line
+	6450 2700 6350 2700
+Wire Wire Line
+	6350 2700 6350 2800
+Wire Wire Line
+	5950 2500 6450 2500
+Wire Wire Line
+	5950 2600 6450 2600
 $EndSCHEMATC

Commit message: correcciones agregadas
Connections:
- net VCC renamed +5V
Changed lines of the file:
@@
 AR Path="/60DC5AA5/6102AF98" Ref="J?"  Part="1"
 AR Path="/6101F213/6102AF98" Ref="J4"  Part="1"
-F 0 "J4" H 5700 4817 50  0000 C CNN
-F 1 "Conn_02x24_Counter_Clockwise" H 5700 4726 50  0000 C CNN
+F 0 "J4" H 5700 2200 50  0000 C CNN
+F 1 "Conn_02x24_Counter_Clockwise" H 5700 2100 50  0000 C CNN
 F 2 "Package_DIP:DIP-48_W15.24mm_LongPads" H 5650 3500 50  0001 C CNN
 F 3 "~" H 5650 3500 50  0001 C CNN
@@
 	1    0    0    -1
 $EndComp
-Text HLabel 5950 2400 2    50   Input ~ 0
+Text HLabel 5950 2400 1    50   Input ~ 0
 VCC
 Text HLabel 5950 2700 2    50   BiDi ~ 0
@@
 Text HLabel 5950 4700 2    50   BiDi ~ 0
 M3
-Text HLabel 5450 2400 0    50   Input ~ 0
+Text HLabel 5450 2400 1    50   Input ~ 0
 GND
 Text HLabel 5450 2500 0    50   BiDi ~ 0
@@
 Wire Notes Line
 	4700 4950 4700 2000
-Text Notes 4750 4850 0    50   ~ 10
+Text Notes 6650 4300 0    50   ~ 10
 Conector FPGA
 $Comp
@@
 Wire Wire Line
 	5950 2600 6450 2600
+$Comp
+L power:+5V #PWR?
+U 1 1 611C0517
+P 6400 2400
+AR Path="/60DC5AA5/611C0517" Ref="#PWR?"  Part="1"
+AR Path="/6101F213/611C0517" Ref="#PWR0116"  Part="1"
+F 0 "#PWR0116" H 6400 2250 50  0001 C CNN
+F 1 "+5V" H 6415 2573 50  0000 C CNN
+F 2 "" H 6400 2400 50  0001 C CNN
+F 3 "" H 6400 2400 50  0001 C CNN
+	1    6400 2400
+	1    0    0    -1
+$EndComp
+Wire Wire Line
+	6400 2400 5950 2400
+$Comp
+L power:GND #PWR?
+U 1 1 611C601A
+P 5150 2450
+AR Path="/60DC5AA5/611C601A" Ref="#PWR?"  Part="1"
+AR Path="/611C601A" Ref="#PWR?"  Part="1"
+AR Path="/6101F213/611C601A" Ref="#PWR0126"  Part="1"
+F 0 "#PWR0126" H 5150 2200 50  0001 C CNN
+F 1 "GND" H 5155 2277 50  0000 C CNN
+F 2 "" H 5150 2450 50  0001 C CNN
+F 3 "" H 5150 2450 50  0001 C CNN
+	1    5150 2450
+	1    0    0    -1
+$EndComp
+Wire Wire Line
+	5450 2400 5150 2400
+Wire Wire Line
+	5150 2400 5150 2450
 $EndSCHEMATC
